Commit message: Initial commit: Pick and place ROS 2 setup and scripts

File: src/my_pick_and_place/urdf/ur5e_dexhand.xacro (robot description, xacro)
@@ -122,3 +122,113 @@
     </plugin>
   </gazebo>
+  <ros2_control name="DexHandSystem" type="system">
+    <hardware>
+      <plugin>ign_ros2_control/IgnitionSystem</plugin>
+    </hardware>
+    <joint name="R_Index_Pitch">
+      <command_interface name="position"/>
+      <state_interface name="position"/>
+      <state_interface name="velocity"/>
+    </joint>
+    <joint name="R_Middle_Pitch">
+      <command_interface name="position"/>
+      <state_interface name="position"/>
+      <state_interface name="velocity"/>
+    </joint>
+    <joint name="R_Ring_Pitch">
+      <command_interface name="position"/>
+      <state_interface name="position"/>
+      <state_interface name="velocity"/>
+    </joint>
+    <joint name="R_Pinky_Pitch">
+      <command_interface name="position"/>
+      <state_interface name="position"/>
+      <state_interface name="velocity"/>
+    </joint>
+    <joint name="R_Index_Flexor">
+      <command_interface name="position"/>
+      <state_interface name="position"/>
+      <state_interface name="velocity"/>
+    </joint>
+    <joint name="R_Middle_Flexor">
+      <command_interface name="position"/>
+      <state_interface name="position"/>
+      <state_interface name="velocity"/>
+    </joint>
+    <joint name="R_Ring_Flexor">
+      <command_interface name="position"/>
+      <state_interface name="position"/>
+      <state_interface name="velocity"/>
+    </joint>
+    <joint name="R_Pinky_Flexor">
+      <command_interface name="position"/>
+      <state_interface name="position"/>
+      <state_interface name="velocity"/>
+    </joint>
+    <joint name="R_Index_DIP">
+      <command_interface name="position"/>
+      <state_interface name="position"/>
+      <state_interface name="velocity"/>
+    </joint>
+    <joint name="R_Middle_DIP">
+      <command_interface name="position"/>
+      <state_interface name="position"/>
+      <state_interface name="velocity"/>
+    </joint>
+    <joint name="R_Ring_DIP">
+      <command_interface name="position"/>
+      <state_interface name="position"/>
+      <state_interface name="velocity"/>
+    </joint>
+    <joint name="R_Pinky_DIP">
+      <command_interface name="position"/>
+      <state_interface name="position"/>
+      <state_interface name="velocity"/>
+    </joint>
+    <joint name="R_Thumb_Yaw">
+      <command_interface name="position"/>
+      <state_interface name="position"/>
+      <state_interface name="velocity"/>
+    </joint>
+    <joint name="R_Thumb_Roll">
+      <command_interface name="position"/>
+      <state_interface name="position"/>
+      <state_interface name="velocity"/>
+    </joint>
+    <joint name="R_Thumb_Flexor">
+      <command_interface name="position"/>
+      <state_interface name="position"/>
+      <state_interface name="velocity"/>
+    </joint>
+    <joint name="R_Thumb_DIP">
+      <command_interface name="position"/>
+      <state_interface name="position"/>
+      <state_interface name="velocity"/>
+    </joint>
+    <joint name="R_Index_Yaw">
+      <command_interface name="position"/>
+      <state_interface name="position"/>
+      <state_interface name="velocity"/>
+    </joint>
+    <joint name="R_Middle_Yaw">
+      <command_interface name="position"/>
+      <state_interface name="position"/>
+      <state_interface name="velocity"/>
+    </joint>
+    <joint name="R_Ring_Yaw">
+      <command_interface name="position"/>
+      <state_interface name="position"/>
+      <state_interface name="velocity"/>
+    </joint>
+    <joint name="R_Pinky_Yaw">
+      <command_interface name="position"/>
+      <state_interface name="position"/>
+      <state_interface name="velocity"/>
+    </joint>
+    <joint name="R_Thumb_Pitch">
+      <command_interface name="position"/>
+      <state_interface name="position"/>
+      <state_interface name="velocity"/>
+    </joint>
+  </ros2_control>
 </robot>

Commit message: Update mobile base pose and initial arm posture for apple simulation

File: src/my_pick_and_place/urdf/ur5e_dexhand.xacro (robot description, xacro)
@@ -33,8 +33,9 @@
     </inertial>
   </link>
+  <!-- MOVED ROBOT BESIDE APPLES (X=0.8m, Y=-0.8m) AND ROTATED 90 DEGREES (Yaw=1.5708) -->
   <joint name="base_footprint_joint" type="fixed">
     <parent link="base_footprint"/>
     <child link="mobile_base_link"/>
-    <origin xyz="0 0 0.0" rpy="0 0 0"/>
+    <origin xyz="0.8 -0.8 0.0" rpy="0 0 1.5708"/>
   </joint>
   <!-- Drive Wheels -->
@@ -71,5 +72,5 @@
     <parent link="mobile_base_link"/><child link="caster_back"/><origin xyz="-0.3 0 0.06" rpy="0 0 0"/>
   </joint>
-  <!-- Include UR Robot -->
+  <!-- Include UR Robot with Horizontal Arm Pose -->
   <xacro:include filename="$(find ur_description)/urdf/ur_macro.xacro"/>
   <xacro:ur_robot
@@ -86,5 +87,5 @@
     generate_ros2_control_tag="$(arg generate_ros2_control_tag)"
     sim_ignition="$(arg sim_ignition)"
-    initial_positions="${dict(shoulder_pan_joint=0.0, shoulder_lift_joint=-1.5708, elbow_joint=0.0, wrist_1_joint=-1.5708, wrist_2_joint=0.0, wrist_3_joint=0.0)}"
+    initial_positions="${dict(shoulder_pan_joint=0.0, shoulder_lift_joint=-1.5708, elbow_joint=1.5708, wrist_1_joint=-1.5708, wrist_2_joint=-1.5708, wrist_3_joint=0.0)}"
   >
     <origin xyz="0 0 0.285" rpy="0 0 0"/>
@@ -114,13 +115,4 @@
       <child_frame_id>base_footprint</child_frame_id>
     </plugin>
-    <!-- DetachableJoint disabled, switching to real friction-based grasping
-    <plugin filename="ignition-gazebo-detachable-joint-system" name="ignition::gazebo::systems::DetachableJoint">
-      <parent_link>wrist_3_link</parent_link>
-      <child_model>red_block</child_model>
-      <child_link>block_link</child_link>
-      <attach_topic>/attach</attach_topic>
-      <detach_topic>/detach</detach_topic>
-    </plugin>
-    -->
   </gazebo>
   <ros2_control name="DexHandSystem" type="system">

Commit message: Add gripper camera sensor and VLM fragility scoring node

File: src/my_pick_and_place/urdf/ur5e_dexhand.xacro (robot description, xacro)
@@ -98,4 +98,52 @@
     <origin xyz="0 0 0" rpy="0 0 0"/>
   </joint>
+  <!-- Gripper Camera -->
+<link name="gripper_camera_link">
+  <visual>
+    <geometry>
+      <box size="0.04 0.04 0.02"/>
+    </geometry>
+  </visual>
+  <collision>
+    <geometry>
+      <box size="0.04 0.04 0.02"/>
+    </geometry>
+  </collision>
+  <inertial>
+    <mass value="0.05"/>
+    <inertia
+      ixx="0.00001"
+      ixy="0.0"
+      ixz="0.0"
+      iyy="0.00001"
+      iyz="0.0"
+      izz="0.00001"/>
+  </inertial>
+</link>
+<joint name="dexhand_to_camera" type="fixed">
+  <parent link="dexhand_base_link"/>
+  <child link="gripper_camera_link"/>
+  <origin xyz="0.0 -0.06 0.08" rpy="0 0 0"/>
+</joint>
+<gazebo reference="gripper_camera_link">
+  <sensor name="gripper_camera_sensor" type="camera">
+    <always_on>true</always_on>
+    <visualize>true</visualize>
+    <update_rate>30</update_rate>
+    <camera>
+      <horizontal_fov>1.047</horizontal_fov>
+      <image>
+        <width>640</width>
+        <height>480</height>
+        <format>R8G8B8</format>
+      </image>
+      <clip>
+        <near>0.05</near>
+        <far>5.0</far>
+      </clip>
+    </camera>
+    <topic>/gripper_camera</topic>
+  </sensor>
+</gazebo>
   <!-- Gazebo Control Plugins -->
   <gazebo>

Commit message: Update apple SDF models and add full layer grasp script

File: src/my_pick_and_place/urdf/ur5e_dexhand.xacro (robot description, xacro)
@@ -37,5 +37,5 @@
     <parent link="base_footprint"/>
     <child link="mobile_base_link"/>
-    <origin xyz="0.8 -0.8 0.0" rpy="0 0 1.5708"/>
+    <origin xyz="1.375 -0.55 0.0" rpy="0 0 1.5708"/>
   </joint>
   <!-- Drive Wheels -->

Commit message: Remove stale hardcoded offset between base_footprint and the arm mount
base_footprint_joint carried a leftover (1.375, -0.55, +90deg) fixed
transform from before teleport-based positioning existed. teleport()
moves base_footprint to DELIVERY_ROBOT_X/Y/YAW, but the real arm mount
(mobile_base_link) sat over a meter away from that point and rotated an
extra 90 degrees on top -- silently, since it's baked into the URDF and
neither world_to_local() nor solve_ik() knew about it. That put the
apple target behind/beside the real shoulder position instead of in
front of it, forcing the contorted reach-backward IK solutions seen all
session regardless of station tuning. Zeroing the offset makes
base_footprint and the arm mount coincide, matching what the Python
coordinate math already assumed.

File: src/my_pick_and_place/urdf/ur5e_dexhand.xacro (robot description, xacro)
@@ -33,9 +33,17 @@
     </inertial>
   </link>
-  <!-- MOVED ROBOT BESIDE APPLES (X=0.8m, Y=-0.8m) AND ROTATED 90 DEGREES (Yaw=1.5708) -->
+  <!-- Positioning is done dynamically at runtime by teleporting base_footprint (see
+       teleport() / DELIVERY_ROBOT_X/Y/YAW in full_layer_grasp.py). This joint must
+       stay at zero offset, or the real arm mount silently drifts away from wherever
+       the Python math thinks the robot is. It used to carry a hardcoded (1.375, -0.55,
+       +90deg) offset from before teleport-based positioning existed; that stale offset
+       was never accounted for anywhere in world_to_local()/solve_ik(), which is why
+       the arm kept reaching from the "wrong side" no matter what station or IK
+       heuristic was tried: the self-checks were all internally consistent with the
+       wrong physical frame.-->
   <joint name="base_footprint_joint" type="fixed">
     <parent link="base_footprint"/>
     <child link="mobile_base_link"/>
-    <origin xyz="1.375 -0.55 0.0" rpy="0 0 1.5708"/>
+    <origin xyz="0 0 0.0" rpy="0 0 0"/>
   </joint>
   <!-- Drive Wheels -->
