Commit message: Add optional fingertip force sensors (tactile:=true), off by default
Joint effort is a torque that saturates at 1.5Nm, so a firm grip and a crushing grip read
the same, and contact has to be inferred from a noise threshold measured in free air each
run. ur5e_dexhand.xacro can now put a force_torque sensor in each fingertip joint, and
apple_world.world loads the ForceTorque and Contact systems (inert while no sensor is
declared). Verified with xacro: the default build has 0 force_torque blocks, tactile:=true
has 5; both parse. start_everything.sh takes a 'tactile' argument that builds that robot
and bridges the five sensor topics; without it the robot, world and topics are exactly
what picked all ten apples. tactile_check.py prints fingertip force next to joint effort
so the sensors can be validated before any control reads them.

Co-Authored-By: Claude Opus 5 <noreply@anthropic.com>

File: src/my_pick_and_place/urdf/ur5e_dexhand.xacro (robot description, xacro)
@@ -15,4 +15,32 @@
   <xacro:arg name="generate_ros2_control_tag" default="true"/>
   <xacro:arg name="sim_ignition" default="true"/>
+  <!-- Fingertip force sensing, OFF by default so every existing launch produces exactly
+       the robot that picked all ten apples. With tactile:=true, each fingertip joint gets
+       a force_torque sensor: a load cell in the tip, reading contact force in newtons.
+       Needed because joint effort (what the grasp reads today) is a torque that saturates
+       at 1.5Nm, so a firm grip and a crushing grip read the same. -->
+  <xacro:arg name="tactile" default="false"/>
+  <xacro:property name="tactile_rate" value="100"/>
+  <xacro:if value="$(arg tactile)">
+    <xacro:macro name="fingertip_ft" params="joint sensor">
+      <gazebo reference="${joint}">
+        <sensor name="${sensor}" type="force_torque">
+          <always_on>1</always_on>
+          <update_rate>${tactile_rate}</update_rate>
+          <visualize>false</visualize>
+          <force_torque>
+            <!-- Report in the child (fingertip) frame: that is where contact happens. -->
+            <frame>child</frame>
+            <measure_direction>parent_to_child</measure_direction>
+          </force_torque>
+        </sensor>
+      </gazebo>
+    </xacro:macro>
+    <xacro:fingertip_ft joint="R_Index_DIP"  sensor="index_tip_ft"/>
+    <xacro:fingertip_ft joint="R_Middle_DIP" sensor="middle_tip_ft"/>
+    <xacro:fingertip_ft joint="R_Ring_DIP"   sensor="ring_tip_ft"/>
+    <xacro:fingertip_ft joint="R_Pinky_DIP"  sensor="pinky_tip_ft"/>
+    <xacro:fingertip_ft joint="R_Thumb_DIP"  sensor="thumb_tip_ft"/>
+  </xacro:if>
   <link name="base_footprint"/>
   <!-- Mobile Base -->

Commit message: Fix the tactile baseline per finger, track peaks, and drop the sensor rate to 50Hz
The single hand-wide baseline was taken before four of the five sensors had published, so
only the index finger read zero at rest. Each finger now zeroes on its own first reading.
The checker also keeps the highest force and effort seen per finger and prints them every
ten samples, so a brief contact during a grasp is still visible afterwards. Sensor rate
100Hz -> 50Hz: at 100Hz the simulation ran 0.070x real time against about 0.11x without
sensors, and this project has twice been bitten by timing changing the grasp.

Co-Authored-By: Claude Opus 5 <noreply@anthropic.com>

File: src/my_pick_and_place/urdf/ur5e_dexhand.xacro (robot description, xacro)
@@ -21,5 +21,8 @@
        at 1.5Nm, so a firm grip and a crushing grip read the same. -->
   <xacro:arg name="tactile" default="false"/>
-  <xacro:property name="tactile_rate" value="100"/>
+  <!-- 50Hz, not 100: at 100 the simulation dropped from about 0.11x to 0.070x real
+       time, and this project has already been bitten twice by timing changing the
+       grasp. 50Hz is still 20 samples per closing step. -->
+  <xacro:property name="tactile_rate" value="50"/>
   <xacro:if value="$(arg tactile)">
     <xacro:macro name="fingertip_ft" params="joint sensor">

Commit message: Contact sensors on all 15 finger segments (tactile), and a 'fragility' launch switch
The fingertip force_torque sensors report joint reaction force (about 100N on the thumb
holding a 4N apple) and see only the tip link, so the 12cm apple held on inner segments
read 0N. tactile:=true now also adds a contact sensor on each proximal, middle and tip
segment, publishing /tactile/<finger>_<segment>; collision names were taken from the
URDF->SDF conversion and all 15 sensors survive it with their topics. The default build
still has zero sensors. start_everything.sh bridges all 20 sensor topics in one process,
and 'fragility' loads apple_world_fragility.world (aborting if it is missing); with no
arguments the world path and robot are exactly as before.

Co-Authored-By: Claude Opus 5 <noreply@anthropic.com>

File: src/my_pick_and_place/urdf/ur5e_dexhand.xacro (robot description, xacro)
@@ -45,4 +45,37 @@
     <xacro:fingertip_ft joint="R_Pinky_DIP"  sensor="pinky_tip_ft"/>
     <xacro:fingertip_ft joint="R_Thumb_DIP"  sensor="thumb_tip_ft"/>
+    <!-- Contact sensors on EVERY finger segment, not just the tips. The force_torque
+         sensors above report the joint's reaction force (about 100N on the thumb while
+         holding a 4N apple) and only see the tip link, so the 12cm apple, held on the
+         inner segments, read 0N while it was held. A contact sensor reports which segment
+         touches what, where, and how deep. Collision names are what the URDF->SDF
+         conversion produces for these links (checked with ign sdf -p). -->
+    <xacro:macro name="segment_contact" params="link topic">
+      <gazebo reference="${link}">
+        <sensor name="${topic}_contact" type="contact">
+          <always_on>1</always_on>
+          <update_rate>${tactile_rate}</update_rate>
+          <topic>/tactile/${topic}</topic>
+          <contact>
+            <collision>${link}_collision</collision>
+          </contact>
+        </sensor>
+      </gazebo>
+    </xacro:macro>
+    <xacro:segment_contact link="Index_Knuckle_1"  topic="index_proximal"/>
+    <xacro:segment_contact link="Index_Middle_1"   topic="index_middle"/>
+    <xacro:segment_contact link="Index_Tip_1"      topic="index_tip"/>
+    <xacro:segment_contact link="Middle_Knuckle_1" topic="middle_proximal"/>
+    <xacro:segment_contact link="Middle_Middle_1"  topic="middle_middle"/>
+    <xacro:segment_contact link="Midle_Tip_1"      topic="middle_tip"/>
+    <xacro:segment_contact link="Ring_Knuckle_1"   topic="ring_proximal"/>
+    <xacro:segment_contact link="Ring_Middle_1"    topic="ring_middle"/>
+    <xacro:segment_contact link="Ring_Tip_1"       topic="ring_tip"/>
+    <xacro:segment_contact link="Pinky_Knuckle_1"  topic="pinky_proximal"/>
+    <xacro:segment_contact link="Pinky_Middle_1"   topic="pinky_middle"/>
+    <xacro:segment_contact link="Pinky_Tip_1"      topic="pinky_tip"/>
+    <xacro:segment_contact link="Thumb_Knuckle_1"  topic="thumb_proximal"/>
+    <xacro:segment_contact link="Thumb_Middle_1"   topic="thumb_middle"/>
+    <xacro:segment_contact link="Thumb_Tip_1"      topic="thumb_tip"/>
   </xacro:if>
   <link name="base_footprint"/>
