Commit message: Fix dead fingertip joints: mimic tags pointed at non-existent master joints
All five DIP (fingertip) joints were declared as mimic joints slaved to
masters named without the R_ prefix -- Index_Flexor, Middle_Flexor,
Ring_Flexor, Pinky_Flexor, Thumb_Flexor -- none of which exist. Every
real joint in this hand carries the R_ prefix (R_Index_Flexor etc.), so
each fingertip was chained to a phantom master and could never move. As
mimic joints they also could not be commanded directly, so the positions
the grasp code sends for them were silently discarded.

Measured consequence: the index fingertip sits 16.74cm from the wrist
open and 16.68cm at full closure -- it travels 0.6mm. The fingers only
pivot at the knuckle and stay rigid, so thumb-to-index span only closes
from 15.38cm to 12.00cm, leaving an 8.00cm apple with 2cm of air on
either side. That is why only R_Middle ever registered contact (its
knuckle rotation grazes the apple) while the other four read pure noise,
regardless of height, station, or closing schedule -- and why no grasp
has ever succeeded in this project.

Removing the mimic tags rather than re-pointing them at the real masters,
since the code already commands each DIP explicitly at 0.8x pitch and the
controller lists them; re-pointing would leave a mimic-vs-command
conflict.

Co-Authored-By: Claude Opus 5 <noreply@anthropic.com>

File: src/dexhandv2_description/urdf/dexhandv2_right.urdf (robot description, URDF)
Before this commit: robot dexhandv2_right, 22 links, 21 joints
Joints:
- joint R_Index_DIP: mimic joint=Index_Flexor multiplier=1 offset=0 -> (none)
- joint R_Middle_DIP: mimic joint=Middle_Flexor multiplier=1 offset=0 -> (none)
- joint R_Pinky_DIP: mimic joint=Pinky_Flexor multiplier=1 offset=0 -> (none)
- joint R_Ring_DIP: mimic joint=Ring_Flexor multiplier=1 offset=0 -> (none)
- joint R_Thumb_DIP: mimic joint=Thumb_Flexor multiplier=1 offset=0 -> (none)

Commit message: Cap finger joint effort at 1.5Nm so the hand cannot slam the apple away
Every one of the 21 finger joints allowed 100Nm. For a fingertip that is
enormous -- a human finger manages a few Nm -- so however slowly the
commands are stepped, the moment a finger meets resistance the position
controller can drive up to 100Nm into a 0.54kg apple.

The measurements show exactly that happening. In the best attempt this
run (5/5 contacts, wrist within 0.019m, palm 6deg from parallel) the
closing peaks were R_Ring 8.585Nm, R_Pinky 7.829Nm, R_Thumb 6.491Nm --
and immediately afterwards the holding force read R_Ring 0.04, R_Thumb
0.05. The fingers squeezed hard enough to squirt the apple out from
between them, then finished closing on empty air. Slowing the command
steps cannot fix that; the joint needs a physical ceiling.

Capping at 1.5Nm still comfortably exceeds the roughly 0.5Nm needed to
hold this apple's weight through friction, while removing the headroom
that lets a finger launch it.

Co-Authored-By: Claude Opus 5 <noreply@anthropic.com>

File: src/dexhandv2_description/urdf/dexhandv2_right.urdf (robot description, URDF)
Before this commit: robot dexhandv2_right, 22 links, 21 joints
Joints:
- joint R_Index_DIP: limit lower=0.0 upper=1.047198 effort=100 velocity=100 -> lower=0.0 upper=1.047198 effort=1.5 velocity=100
- joint R_Index_Flexor: limit lower=0.0 upper=1.047198 effort=100 velocity=100 -> lower=0.0 upper=1.047198 effort=1.5 velocity=100
- joint R_Index_Pitch: limit lower=0.0 upper=1.308997 effort=100 velocity=100 -> lower=0.0 upper=1.308997 effort=1.5 velocity=100
- joint R_Index_Yaw: limit lower=-0.349066 upper=0.349066 effort=100 velocity=100 -> lower=-0.349066 upper=0.349066 effort=1.5 velocity=100
- joint R_Middle_DIP: limit lower=0.0 upper=1.047198 effort=100 velocity=100 -> lower=0.0 upper=1.047198 effort=1.5 velocity=100
- joint R_Middle_Flexor: limit lower=0.0 upper=1.047198 effort=100 velocity=100 -> lower=0.0 upper=1.047198 effort=1.5 velocity=100
- joint R_Middle_Pitch: limit lower=0.0 upper=1.308997 effort=100 velocity=100 -> lower=0.0 upper=1.308997 effort=1.5 velocity=100
- joint R_Middle_Yaw: limit lower=-0.349066 upper=0.349066 effort=100 velocity=100 -> lower=-0.349066 upper=0.349066 effort=1.5 velocity=100
- joint R_Pinky_DIP: limit lower=0.0 upper=1.047198 effort=100 velocity=100 -> lower=0.0 upper=1.047198 effort=1.5 velocity=100
- joint R_Pinky_Flexor: limit lower=0.0 upper=1.047198 effort=100 velocity=100 -> lower=0.0 upper=1.047198 effort=1.5 velocity=100
- joint R_Pinky_Pitch: limit lower=0.0 upper=1.308997 effort=100 velocity=100 -> lower=0.0 upper=1.308997 effort=1.5 velocity=100
- joint R_Pinky_Yaw: limit lower=-0.349066 upper=0.349066 effort=100 velocity=100 -> lower=-0.349066 upper=0.349066 effort=1.5 velocity=100
- joint R_Ring_DIP: limit lower=0.0 upper=1.047198 effort=100 velocity=100 -> lower=0.0 upper=1.047198 effort=1.5 velocity=100
- joint R_Ring_Flexor: limit lower=0.0 upper=1.047198 effort=100 velocity=100 -> lower=0.0 upper=1.047198 effort=1.5 velocity=100
- joint R_Ring_Pitch: limit lower=0.0 upper=1.308997 effort=100 velocity=100 -> lower=0.0 upper=1.308997 effort=1.5 velocity=100
- joint R_Ring_Yaw: limit lower=-0.349066 upper=0.349066 effort=100 velocity=100 -> lower=-0.349066 upper=0.349066 effort=1.5 velocity=100
- joint R_Thumb_DIP: limit lower=0.0 upper=1.047198 effort=100 velocity=100 -> lower=0.0 upper=1.047198 effort=1.5 velocity=100
- joint R_Thumb_Flexor: limit lower=0.0 upper=1.047198 effort=100 velocity=100 -> lower=0.0 upper=1.047198 effort=1.5 velocity=100
- joint R_Thumb_Pitch: limit lower=0.0 upper=1.047198 effort=100 velocity=100 -> lower=0.0 upper=1.047198 effort=1.5 velocity=100
- joint R_Thumb_Roll: limit lower=-0.349066 upper=0.349066 effort=100 velocity=100 -> lower=-0.349066 upper=0.349066 effort=1.5 velocity=100
- joint R_Thumb_Yaw: limit lower=-0.523599 upper=0.523599 effort=100 velocity=100 -> lower=-0.523599 upper=0.523599 effort=1.5 velocity=100
